File: Kicad/power_meter_coin/power_meter_coin.kicad_pcb (KiCad board)
At the start: 2 copper layers, 41 x 41 mm, 15 parts, among them IC1 ATTINY84-S, P1 CONN_02X03, P2 CONN_01X03, U1 LM1117

Commit message: ordered version PCB
Other:
- board text added: "3v3"
- board text added: "Vin"
